Commit message: finished

File: body.urdf (robot description, URDF)
Before this commit: robot robot, 2 links, 1 joints
Links:
- removed link Leg
- added link BackLeg, mass 1; collision box size=1 1 1; visual box size=1 1 1
- added link FrontLeg, mass 1; collision box size=1 1 1; visual box size=1 1 1
Joints:
- removed joint Torso_Leg
- added joint BackLeg_Torso: type revolute, parent BackLeg, child Torso, origin xyz=0 1 1 rpy=0 0 0, axis 0 1 0, limit lower=-3.14159 upper=3.14159 effort=0.0 velocity=0.0
- added joint Torso_FrontLeg: type revolute, parent Torso, child FrontLeg, origin xyz=0 1 0 rpy=0 0 0, axis 0 1 0, limit lower=-3.14159 upper=3.14159 effort=0.0 velocity=0.0

Commit message: sensor touch

File: body.urdf (robot description, URDF)
Before this commit: robot robot, 3 links, 2 joints
Joints:
- joint BackLeg_Torso: origin xyz=0 1 1 rpy=0 0 0 -> xyz=1 0 1 rpy=0 0 0
- joint Torso_FrontLeg: origin xyz=0 1 0 rpy=0 0 0 -> xyz=1 0 0 rpy=0 0 0

Commit message: more

File: body.urdf (robot description, URDF)
Before this commit: robot robot, 3 links, 2 joints
Joints:
- removed joint BackLeg_Torso
- added joint Torso_BackLeg: type revolute, parent Torso, child BackLeg, origin xyz=0.5 0.5 1 rpy=0 0 0, axis 0 1 0, limit lower=-3.14159 upper=3.14159 effort=0.0 velocity=0.0
- joint Torso_FrontLeg: origin xyz=1 0 0 rpy=0 0 0 -> xyz=0 -0.5 1 rpy=0 0 0

Commit message: motors branch

File: body.urdf (robot description, URDF)
Before this commit: robot robot, 3 links, 2 joints
Joints:
- joint Torso_BackLeg: origin xyz=0.5 0.5 1 rpy=0 0 0 -> xyz=2 0 1 rpy=0 0 0
- joint Torso_FrontLeg: origin xyz=0 -0.5 1 rpy=0 0 0 -> xyz=1 0 1 rpy=0 0 0

Commit message: final

File: body.urdf (robot description, URDF)
Before this commit: robot robot, 3 links, 2 joints
Links:
- removed link BackLeg
- removed link FrontLeg
- removed link Torso
- added link Arm1, mass 1; collision box size=0.5 1 0.1; visual box size=0.5 1 0.1
- added link Arm2, mass 1; collision box size=0.5 1 0.1; visual box size=0.5 1 0.1
- added link Limb1, mass 1; collision box size=1 0.5 1; visual box size=1 0.5 1
- added link Limb2, mass 1; collision box size=1 0.5 1; visual box size=1 0.5 1
- added link Main, mass 1; collision box size=1 1 1; visual box size=1 1 1
- added link TopHat, mass 1; collision box size=0.1 0.1 1; visual box size=0.1 0.1 1
- added link Up1, mass 1; collision box size=0.5 0.1 1.5; visual box size=0.5 0.1 1.5
- added link Up2, mass 1; collision box size=0.5 0.1 1.5; visual box size=0.5 0.1 1.5
Joints:
- removed joint Torso_BackLeg
- removed joint Torso_FrontLeg
- added joint Arm1_Up1: type revolute, parent Arm1, child Up1, origin xyz=0 1 0 rpy=0 0 0, axis 0 1 0, limit lower=-3.14159 upper=3.14159 effort=0.0 velocity=0.0
- added joint Arm1_Up2: type revolute, parent Arm1, child Up2, origin xyz=0 -2 0 rpy=0 0 0, axis 0 1 0, limit lower=-3.14159 upper=3.14159 effort=0.0 velocity=0.0
- added joint Main_Arm1: type revolute, parent Main, child Arm1, origin xyz=1.5 0.5 1.5 rpy=0 0 0, axis 0 1 0, limit lower=-3.14159 upper=3.14159 effort=0.0 velocity=0.0
- added joint Main_Arm2: type revolute, parent Main, child Arm2, origin xyz=1.5 -0.5 1.5 rpy=0 0 0, axis 0 1 0, limit lower=-3.14159 upper=3.14159 effort=0.0 velocity=0.0
- added joint Main_Limb1: type revolute, parent Main, child Limb1, origin xyz=2 0 1 rpy=0 0 0, axis 0 1 0, limit lower=-3.14159 upper=3.14159 effort=0.0 velocity=0.0
- added joint Main_Limb2: type revolute, parent Main, child Limb2, origin xyz=1 0 1 rpy=0 0 0, axis 0 1 0, limit lower=-3.14159 upper=3.14159 effort=0.0 velocity=0.0
- added joint Main_TopHat: type revolute, parent Main, child TopHat, origin xyz=1.5 0 2 rpy=0 0 0, axis 0 1 0, limit lower=-3.14159 upper=3.14159 effort=0.0 velocity=0.0
